File: Big Daddy-2025-04-11_172858/Big Daddy-2025-04-11_172858/Big Daddy.kicad_sch (KiCad schematic)
At the start: 0 parts

Commit message: all the bs
Other:
- sheet Connectors ports: added TSSI_Green_in, TSSI_Green_out, TSSI_Red_in, TSSI_Red_out; removed SSOK, TSAL_GND, TSAL_PWR
- sheet Fusing ports: added 12V_in; removed none
- sheet High Voltage ports: added 12V_in, TSSI_Fault, TSSI_Green_in, TSSI_Green_out, TSSI_Red_in, TSSI_Red_out; removed TSAL_GND, TSAL_PWR
- sheet Latching ports: added 12V_in; removed LOOP_IN
- sheet Microcontrolller ports: added TSSI_Fault, Traction_Toggle; removed VICOR_Tempt?
