File: Big Daddy-2025-04-11_172858/Big Daddy-2025-04-11_172858/High Voltage.kicad_sch (KiCad schematic)
At the start: 2 parts

Commit message: all the bs
Other:
- sheet TSAL ports: added 12V_in, TSSI_Fault, TSSI_Green_in, TSSI_Green_out, TSSI_Red_in, TSSI_Red_out; removed TSAL_GND, TSAL_PWR
Changed lines of the file:
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@@
-	(wire
-		(pts
-			(xy 186.69 131.572) (xy 189.23 131.572)
-		)
-		(stroke
-			(width 0)
-			(type default)
-		)
-	)
 	(wire
 		(pts
@@
 	(wire
 		(pts
+			(xy 242.57 115.57) (xy 229.616 115.57)
+		)
+		(stroke
+			(width 0)
+			(type default)
+		)
+	)
+	(wire
+		(pts
 			(xy 186.944 67.31) (xy 188.976 67.31)
 		)
@@
 	(wire
 		(pts
-			(xy 186.436 125.222) (xy 189.23 125.222)
+			(xy 242.57 111.76) (xy 229.616 111.76)
+		)
+		(stroke
+			(width 0)
+			(type default)
+		)
+	)
+	(wire
+		(pts
+			(xy 229.616 125.73) (xy 242.57 125.73)
 		)
 		(stroke
@@
 	(wire
 		(pts
+			(xy 229.616 130.81) (xy 241.3 130.81)
+		)
+		(stroke
+			(width 0)
+			(type default)
+		)
+	)
+	(wire
+		(pts
 			(xy 154.178 58.674) (xy 154.178 92.202)
 		)
@@
 	(wire
 		(pts
+			(xy 243.84 120.65) (xy 229.616 120.65)
+		)
+		(stroke
+			(width 0)
+			(type default)
+		)
+	)
+	(wire
+		(pts
 			(xy 186.69 76.708) (xy 188.976 76.708)
 		)
@@
 		(pts
 			(xy 176.53 112.014) (xy 189.23 112.014)
+		)
+		(stroke
+			(width 0)
+			(type default)
+		)
+	)
+	(wire
+		(pts
+			(xy 229.616 107.95) (xy 236.22 107.95)
 		)
 		(stroke
@@
 		)
 	)
+	(hierarchical_label "TSSI_Green_in"
+		(shape output)
+		(at 243.84 120.65 0)
+		(effects
+			(font
+				(size 1.27 1.27)
+			)
+			(justify left)
+		)
+	)
+	(hierarchical_label "TSSI_Red_out"
+		(shape output)
+		(at 241.3 130.81 0)
+		(effects
+			(font
+				(size 1.27 1.27)
+			)
+			(justify left)
+		)
+	)
+	(hierarchical_label "TSSI_Fault"
+		(shape input)
+		(at 242.57 111.76 0)
+		(effects
+			(font
+				(size 1.27 1.27)
+			)
+			(justify left)
+		)
+	)
+	(hierarchical_label "TSSI_Green_out"
+		(shape output)
+		(at 242.57 125.73 0)
+		(effects
+			(font
+				(size 1.27 1.27)
+			)
+			(justify left)
+		)
+	)
 	(hierarchical_label "Vicor_OUT"
 		(shape output)
@@
 		)
 	)
-	(hierarchical_label "TSAL_GND"
+	(hierarchical_label "12V_in"
+		(shape input)
+		(at 236.22 107.95 0)
+		(effects
+			(font
+				(size 1.27 1.27)
+			)
+			(justify left)
+		)
+	)
+	(hierarchical_label "TSSI_Red_in"
 		(shape output)
-		(at 186.69 131.572 180)
-		(effects
-			(font
-				(size 1.27 1.27)
-			)
-			(justify right)
+		(at 242.57 115.57 0)
+		(effects
+			(font
+				(size 1.27 1.27)
+			)
+			(justify left)
 		)
 	)
@@
 		(shape output)
 		(at 186.944 69.85 180)
-		(effects
-			(font
-				(size 1.27 1.27)
-			)
-			(justify right)
-		)
-	)
-	(hierarchical_label "TSAL_PWR"
-		(shape output)
-		(at 186.436 125.222 180)
 		(effects
 			(font
@@
 			)
 		)
-		(pin "TSAL_GND" output
-			(at 189.23 131.572 180)
-			(effects
-				(font
-					(size 1.27 1.27)
-				)
-				(justify left)
-			)
-		)
-		(pin "TSAL_PWR" output
-			(at 189.23 125.222 180)
-			(effects
-				(font
-					(size 1.27 1.27)
-				)
-				(justify left)
-			)
-		)
 		(pin "HV-" input
 			(at 189.23 112.014 180)
@@
 			)
 		)
+		(pin "TSSI_Red_out" input
+			(at 229.616 130.81 0)
+			(effects
+				(font
+					(size 1.27 1.27)
+				)
+				(justify right)
+			)
+		)
+		(pin "TSSI_Green_out" input
+			(at 229.616 125.73 0)
+			(effects
+				(font
+					(size 1.27 1.27)
+				)
+				(justify right)
+			)
+		)
+		(pin "TSSI_Green_in" input
+			(at 229.616 120.65 0)
+			(effects
+				(font
+					(size 1.27 1.27)
+				)
+				(justify right)
+			)
+		)
+		(pin "TSSI_Red_in" input
+			(at 229.616 115.57 0)
+			(effects
+				(font
+					(size 1.27 1.27)
+				)
+				(justify right)
+			)
+		)
+		(pin "12V_in" input
+			(at 229.616 107.95 0)
+			(effects
+				(font
+					(size 1.27 1.27)
+				)
+				(justify right)
+			)
+		)
+		(pin "TSSI_Fault" input
+			(at 229.616 111.76 0)
+			(effects
+				(font
+					(size 1.27 1.27)
+				)
+				(justify right)
+			)
+		)
