File: Big Daddy-2025-04-11_172858/Big Daddy-2025-04-11_172858/TSAL.kicad_sch (KiCad schematic)
At the start: 21 parts, among them J1 TSSI_Grn I/O, J16 TSSI_Red I/O, Q2 RU1C002UN, Q5 RU1C002UN, U13 LTV-352T, U6 ICM7555xB, U7 IS31LT3360

Commit message: all the bs
Parts:
- removed C12: 100uF, Capacitor_THT:CP_Radial_D10.0mm_P5.00mm, symbol Device:C
- removed C13: .1uF, Capacitor_SMD:C_0603_1608Metric_Pad1.08x0.95mm_HandSolder, symbol Device:C
- removed D9: D_Zener, Diode_SMD:D_SOD-123, symbol Device:D_Zener
- removed L1: 47uH, Inductor_SMD:L_0603_1608Metric_Pad1.05x0.95mm_HandSolder, symbol Device:L
- removed R26, R29: 10k, Resistor_SMD:R_0603_1608Metric_Pad0.98x0.95mm_HandSolder, symbol Device:R_US
- removed R30: 0.15, Resistor_SMD:R_0603_1608Metric_Pad0.98x0.95mm_HandSolder, symbol Device:R_US
- removed U7: IS31LT3360, Package_TO_SOT_SMD:SOT-89-5, symbol Driver_LED:IS31LT3360
- R27: value 15k -> 24k
Connections:
- net 555_OUT: no longer R27.1
- net VDD: now also R27.1, U6.7 (DIS)
- net HV_ON renamed TSSI_Fault
- net INT_12V renamed 12V_in
- net 12V_in: no longer J16.1 (Pin_1), Q2.1 (D)
- new net TSSI_Red_in: J16.1 (Pin_1), Q2.1 (D)
Other:
- note added: "TSSI_Green"
- note added: "TSSI_Red"
- note removed: "*Optional just in case LED Drive does not work"
- note removed: "Change TSAL to TSSI_RED_PWR,"
- note removed: "LED Driver"
- moved on the sheet: J1, J16, Q2, Q5, R27, U6
